Commit message: changed camera position, removed road texture

File: urdf/macros.xacro (robot description, xacro)
@@ -298,5 +298,5 @@
       <origin xyz="0 0 0.25" rpy="0 0 0"/>
       <geometry>
-        <box size="0.033 0.175 0.030"/>
+        <box size="0.033 0.0 0.030"/>
       </geometry>
     </collision>
@@ -320,5 +320,5 @@
     <inertial>
       <mass value="1e-5" />
-      <origin xyz="-2.5 1.5 1.75" rpy="0 .57 -0.57"/>
+      <origin xyz="-0.5 0.0 0.0" rpy="0 .57 -0.57"/>
       <inertia ixx="1e-6" ixy="0" ixz="0" iyy="1e-6" iyz="0" izz="1e-6" />
     </inertial>
@@ -439,5 +439,5 @@
   <!-- camera object -->
   <xacro:unless value="$(optenv DISABLE_GAZEBO_CAMERA false)">
-    <gazebo reference="$(arg robot_name)_camera_link">
+    <gazebo reference="$(arg robot_name)_base_link">
       <sensor type="camera" name="$(arg robot_name)_left_sensor">
         <update_rate>30.0</update_rate>
@@ -467,5 +467,5 @@
           <imageTopicName>image</imageTopicName>
           <cameraInfoTopicName>rgb/camera_info</cameraInfoTopicName>
-          <frameName>$(arg robot_name)_camera_link</frameName>
+          <frameName>$(arg robot_name)_base_link</frameName>
           <hackBaseline>0</hackBaseline><!-- set this to 0.12 for the second camera -->
           <distortionK1>0.0</distortionK1>
